File: ADX KiCAD PCB FILES/ADX.kicad_pcb (KiCad board)
At the start: 2 copper layers, 97.1 x 97 mm, 82 parts, among them CON1 SPK, CON2 MIC, J1 SMA, J1A1 BNC, J2 PJ-102A, Q1 BS170, Q2 BS170, Q3 BS170, Q4 BS170, SW1 UP(BAND), SW2 DOWN(CAL), SW3 TX, U1 CD2003GB_GP, U2 SI535X_Module, U3 74ACT244, U4 uSDX_LPF_BAND_MODULE

Commit message: Refactor
Parts:
- removed C13: 10uF/16V, Capacitor_THT:CP_Radial_D5.0mm_P2.50mm
- removed CX1: , Capacitor_THT:C_Disc_D3.0mm_W1.6mm_P2.50mm
- removed D6: 1N4148, Diode_THT:D_A-405_P2.54mm_Vertical_AnodeUp
- removed the R13 at (107.2, 32.1)
- removed the U1 at (86.2, 55.6)
- added C25: 10n, Capacitor_SMD:C_0805_2012Metric, F.Cu at (228.9, 83.2)
- added C26: 10n, Capacitor_SMD:C_0805_2012Metric, F.Cu at (233.4, 68.1)
- added C27: 10n, Capacitor_SMD:C_0805_2012Metric, F.Cu at (233.4, 71.2)
- added C28: 620p, Capacitor_SMD:C_0805_2012Metric, F.Cu at (233.4, 74.2)
- added D10: 1N4148WS, Diode_SMD:D_SOD-323, F.Cu at (207.4, 97.1)
- added J3: LED, Connector_PinHeader_2.54mm:PinHeader_1x05_P2.54mm_Vertical, F.Cu at (229.5, 87.0)
- added J4: LED_GND, Connector_PinHeader_2.54mm:PinHeader_1x05_P2.54mm_Vertical, F.Cu at (234.2, 87.0)
- added J5: SW, Connector_PinHeader_2.54mm:PinHeader_1x03_P2.54mm_Vertical, F.Cu at (240.8, 85.1)
- added J6: SW_GND, Connector_PinHeader_2.54mm:PinHeader_1x03_P2.54mm_Vertical, F.Cu at (245.5, 85.1)
- added R12: 5.1k, Resistor_SMD:R_0402_1005Metric, F.Cu at (176.3, 85.9)
- added R16: 1k, Resistor_SMD:R_0402_1005Metric, F.Cu at (181.1, 125.0)
- added R16: 1k, Resistor_THT:R_Axial_DIN0204_L3.6mm_D1.6mm_P1.90mm_Vertical, F.Cu at (223.8, 86.3)
- added R17: 1k, Resistor_SMD:R_0402_1005Metric, F.Cu at (181.1, 127.0)
- added R17: 1k, Resistor_THT:R_Axial_DIN0204_L3.6mm_D1.6mm_P1.90mm_Vertical, F.Cu at (223.8, 89.4)
- added R18: 1k, Resistor_THT:R_Axial_DIN0204_L3.6mm_D1.6mm_P1.90mm_Vertical, F.Cu at (223.8, 92.6)
- added R18: 1k, Resistor_SMD:R_0402_1005Metric, F.Cu at (184.0, 119.0)
- added R19: 1k, Resistor_THT:R_Axial_DIN0204_L3.6mm_D1.6mm_P1.90mm_Vertical, F.Cu at (223.8, 95.7)
- added R19: 1k, Resistor_SMD:R_0402_1005Metric, F.Cu at (184.0, 121.0)
- added R20: 1k, Resistor_THT:R_Axial_DIN0204_L3.6mm_D1.6mm_P1.90mm_Vertical, F.Cu at (223.8, 99.8)
- added R20: 1k, Resistor_SMD:R_0402_1005Metric, F.Cu at (184.0, 123.0)
- added U3: CD2003GB_GP, Package_DIP:DIP-16_W7.62mm_Socket_LongPads, F.Cu at (189.2, 115.8)
- C1: value 100uF/16V -> 100u; footprint Capacitor_THT:CP_Radial_D5.0mm_P2.50mm -> Capacitor_SMD:C_1206_3216Metric
- C10, C2, C22, C3, C8, C9: value 100nF -> 100n; footprint Capacitor_THT:C_Disc_D3.0mm_W1.6mm_P2.50mm -> Capacitor_SMD:C_0805_2012Metric
- C11: value 620pF -> 100n; footprint Capacitor_THT:C_Disc_D3.0mm_W1.6mm_P2.50mm -> Capacitor_SMD:C_0805_2012Metric
- C12, C17: value 10nF -> 100n; footprint Capacitor_THT:C_Disc_D3.0mm_W2.0mm_P2.50mm -> Capacitor_SMD:C_0805_2012Metric
- C14, C15: value 100nF -> 10n; footprint Capacitor_THT:C_Disc_D3.0mm_W1.6mm_P2.50mm -> Capacitor_SMD:C_0805_2012Metric
- C16, C24: value 100uF/16V -> 22u; footprint Capacitor_THT:CP_Radial_D5.0mm_P2.50mm -> Capacitor_SMD:C_0805_2012Metric
- C18: value 10uF/16V -> 100n; footprint Capacitor_THT:CP_Radial_D5.0mm_P2.50mm -> Capacitor_SMD:C_0805_2012Metric
- C19, C20, C21, C23: value 100nF -> 22u; footprint Capacitor_THT:C_Disc_D3.0mm_W1.6mm_P2.50mm -> Capacitor_SMD:C_0805_2012Metric
- C4: value 10nF -> 100n; footprint Capacitor_THT:C_Disc_D3.0mm_W1.6mm_P2.50mm -> Capacitor_SMD:C_0805_2012Metric
- C5: value 10nF -> 10n; footprint Capacitor_THT:C_Disc_D3.0mm_W1.6mm_P2.50mm -> Capacitor_SMD:C_0805_2012Metric
- C6: value 100nF -> 470n; footprint Capacitor_THT:C_Disc_D3.0mm_W1.6mm_P2.50mm -> Capacitor_SMD:C_0603_1608Metric
- C7: value 470nF -> 10n; footprint Capacitor_THT:C_Disc_D3.0mm_W1.6mm_P2.50mm -> Capacitor_SMD:C_0805_2012Metric
- D7, D8: value 1N4148 -> 1N4148WS; footprint Diode_THT:D_A-405_P2.54mm_Vertical_KathodeUp -> Diode_SMD:D_SOD-323
- D9: value 1N5817 -> 1N4148WS; footprint Diode_THT:D_A-405_P2.54mm_Vertical_KathodeUp -> Diode_SMD:D_SOD-323
- GND1, TP_D1, TP_G1, TP_S1: value (none) -> ~
- J2: value PJ-102A -> XT60PW-M; footprint digikey-footprints:Barrel_Jack_5.5mmODx2.1mmID_PJ-102A -> XT60PW-M:AMASS_XT60PW-M
- L1: footprint Inductor_THT:L_Toroid_Vertical_L10.0mm_W5.0mm_P5.08mm -> Inductor_SMD:L_0805_2012Metric_Pad1.05x1.20mm_HandSolder
- R1: value 1M -> 10k; footprint Resistor_THT:R_Axial_DIN0204_L3.6mm_D1.6mm_P1.90mm_Vertical -> Resistor_SMD:R_0402_1005Metric
- R10, R11, R15: value 10k -> 1k; footprint Resistor_THT:R_Axial_DIN0204_L3.6mm_D1.6mm_P1.90mm_Vertical -> Resistor_SMD:R_0402_1005Metric
- R13: renamed from R12; footprint Resistor_THT:R_Axial_DIN0204_L3.6mm_D1.6mm_P1.90mm_Vertical -> Resistor_SMD:R_0603_1608Metric
- R14, R4, R5, R6, R8: footprint Resistor_THT:R_Axial_DIN0204_L3.6mm_D1.6mm_P1.90mm_Vertical -> Resistor_SMD:R_0402_1005Metric
- R2: value 4.7k -> 1M; footprint Resistor_THT:R_Axial_DIN0204_L3.6mm_D1.6mm_P1.90mm_Vertical -> Resistor_SMD:R_0402_1005Metric
- R3: value 10k -> 4.7k; footprint Resistor_THT:R_Axial_DIN0204_L3.6mm_D1.6mm_P1.90mm_Vertical -> Resistor_SMD:R_0402_1005Metric
- R7: value 1k -> 5.1k; footprint Resistor_THT:R_Axial_DIN0204_L3.6mm_D1.6mm_P1.90mm_Vertical -> Resistor_SMD:R_0402_1005Metric
- R9: value 1k -> 10k; footprint Resistor_THT:R_Axial_DIN0204_L3.6mm_D1.6mm_P1.90mm_Vertical -> Resistor_SMD:R_0402_1005Metric
- U1: renamed from U3; footprint Package_DIP:DIP-20_W7.62mm_LongPads -> Package_SO:TSSOP-20_4.4x6.5mm_P0.65mm
- moved XA1 179.5 mm to (248.4, 160.0)
- moved C24 163.6 mm to (228.9, 80.2), turned to 0 degrees
- moved C18 162.6 mm to (212.7, 110.0), turned to 0 degrees
- moved D9 156.8 mm to (212.0, 94.7)
- moved C14 153.1 mm to (224.5, 83.2), turned to 0 degrees
- moved C15 152.8 mm to (228.9, 68.1)
- moved C10 140.5 mm to (224.5, 74.2)
- moved C19 140.3 mm to (189.4, 94.9), turned to 0 degrees
- moved C20 138.9 mm to (189.4, 97.9), turned to 0 degrees
- moved C21 138.1 mm to (228.9, 71.2)
- moved SW2 135.3 mm to (216.7, 144.1)
- moved D8 131.9 mm to (207.4, 91.2)
- moved C11 129.3 mm to (224.5, 77.2), turned to 0 degrees
- moved R7 128.1 mm to (225.8, 115.8)
- moved C12 120.0 mm to (224.5, 80.2)
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- renumbered TP8 to TP2, TP2 to TP3, TP3 to TP4, TP4 to TP5, TP7 to TP6
Connections:
- C1 pad 2: GNDPWR -> GND
- C10 pad 1: GNDPWR -> RX_OSC
- C10 pad 2: Net-(C10-Pad2) -> Net-(U3-AM_OSC)
- C11 pad 1: Net-(C11-Pad1) -> Net-(D7-A)
- C11 pad 2: Net-(C11-Pad2) -> GND
- C12 pad 1: RXSW -> GND
- C12 pad 2: GNDPWR -> Net-(U3-FM/AM_SW)
- C14 pad 1: Net-(C13-Pad1) -> RX
- C14 pad 2: GNDPWR -> Net-(Q4-D)
- C15 pad 1: +5V -> GND
- C15 pad 2: GNDPWR -> RXSW
- C16 pad 1: +5V -> +12V
- C16 pad 2: GNDPWR -> GND
- C17 pad 1: Net-(C17-Pad1) -> Net-(D7-A)
- C17 pad 2: RX -> GND
- C18 pad 2: GNDPWR -> GND
- C19 pad 2: GNDPWR -> GND
- C2 pad 2: GNDPWR -> GND
- C20 pad 2: GNDPWR -> GND
- C21 pad 1: Net-(C21-Pad1) -> Net-(D7-A)
- C21 pad 2: RX_OSC -> GND
- C22 pad 1: Net-(C22-Pad1) -> Net-(D7-A)
- C22 pad 2: Net-(C22-Pad2) -> GND
- C23 pad 2: GNDPWR -> GND
- C24 pad 1: +12V -> +5V
- C24 pad 2: GNDPWR -> GND
- C3 pad 1: Net-(C3-Pad1) -> Net-(CON1-R)
- C4 pad 1: Net-(C4-Pad1) -> GND
- C4 pad 2: GNDPWR -> Net-(CON2-R)
- C5 pad 1: FSK -> GND
- C5 pad 2: GNDPWR -> Net-(C5-Pad2)
- C6 pad 1: Net-(C6-Pad1) -> Net-(CON2-R)
- C6 pad 2: GNDPWR -> RXA
- C7 pad 1: Net-(C6-Pad1) -> GND
- C7 pad 2: RXA -> FSK
- C8 pad 1: GNDPWR -> GND
- C8 pad 2: Net-(C13-Pad1) -> +5V
- C9 pad 1: GNDPWR -> Net-(U1-O0a)
- C9 pad 2: Net-(C13-Pad1) -> Net-(D10-K)
- CON1 pad 1: GNDPWR -> GND
- CON1 pad 2: Net-(C3-Pad2) -> Net-(CON1-R)
- CON1 pad 3: Net-(C3-Pad2) -> Net-(CON1-R)
- CON2 pad 1: GNDPWR -> GND
- CON2 pad 2: Net-(C6-Pad1) -> Net-(CON2-R)
- CON2 pad 3: Net-(C6-Pad1) -> Net-(CON2-R)
- D1 pad 1: GNDPWR -> GND
- D2 pad 1: GNDPWR -> GND
- D3 pad 1: GNDPWR -> GND
- D3 pad 2: Net-(D3-Pad2) -> Net-(D3-A)
- D4 pad 1: GNDPWR -> GND
- D4 pad 2: Net-(D4-Pad2) -> Net-(D4-A)
- D5 pad 1: GNDPWR -> GND
- D5 pad 2: Net-(D5-Pad2) -> Net-(D5-A)
- D7 pad 1: Net-(C11-Pad2) -> Net-(D7-K)
- D7 pad 2: Net-(C13-Pad1) -> Net-(D7-A)
- D8 pad 1: Net-(C13-Pad1) -> Net-(D7-A)
- D8 pad 2: Net-(C11-Pad2) -> Net-(D7-K)
- GND1 pad 1: GNDPWR -> GND
- H1 pad 1: GNDPWR -> GND
- H2 pad 1: GNDPWR -> GND
- H3 pad 1: GNDPWR -> GND
- H4 pad 1: GNDPWR -> GND
- J1 pad 2: GNDPWR -> GND
- J1A1 pad 2: GNDPWR -> GND
- J2 pad 2: GNDPWR -> GND
- L1 pad 1: Net-(C11-Pad2) -> Net-(D7-K)
- L1 pad 2: Net-(C13-Pad1) -> Net-(D7-A)
- L2 pad 2: Net-(C13-Pad1) -> Net-(D7-A)
- Q1 pad 2: Net-(C22-Pad1) -> Net-(D10-K)
- Q1 pad 3: GNDPWR -> GND
- Q2 pad 2: Net-(C22-Pad1) -> Net-(D10-K)
- Q2 pad 3: GNDPWR -> GND
- Q3 pad 2: Net-(C22-Pad1) -> Net-(D10-K)
- Q3 pad 3: GNDPWR -> GND
- Q4 pad 1: Net-(C17-Pad1) -> Net-(Q4-D)
- Q4 pad 3: Net-(C11-Pad1) -> Net-(Q4-S)
- R1 pad 1: +3.3V -> +5V
- R1 pad 2: Net-(C3-Pad1) -> SW1
- R10 pad 1: +5V -> Net-(XA1-D10_CS)
- R10 pad 2: SW1 -> Net-(D4-A)
- R11 pad 1: +5V -> Net-(R11-Pad1)
- R11 pad 2: SW2 -> Net-(D5-A)
- R13 pad 1: Net-(C22-Pad1) -> Net-(D10-K)
- R13 pad 2: GNDPWR -> GND
- R14 pad 1: Net-(C21-Pad1) -> Net-(D7-A)
- R14 pad 2: Net-(C13-Pad1) -> Net-(U3-AM_OSC)
- R15 pad 1: +5V -> Net-(Q4-S)
- R15 pad 2: SW3 -> GND
- R2 pad 1: Net-(C3-Pad1) -> +3.3V
- R2 pad 2: GNDPWR -> Net-(C3-Pad2)
- R3 pad 1: Net-(C3-Pad1) -> Net-(C3-Pad2)
- R3 pad 2: Net-(C4-Pad1) -> GND
- R4 pad 1: Net-(C4-Pad1) -> +5V
- R4 pad 2: FSK -> SW2
- R7 pad 1: Net-(R7-Pad1) -> Net-(C3-Pad2)
- R7 pad 2: Net-(D3-Pad2) -> Net-(C5-Pad2)
- R8 pad 1: Net-(R8-Pad1) -> Net-(XA1-D11_MOSI)
- R8 pad 2: Net-(D4-Pad2) -> Net-(D3-A)
- R9 pad 1: Net-(R9-Pad1) -> +5V
- R9 pad 2: Net-(D5-Pad2) -> SW3
- SW1 pad 1: GNDPWR -> GND
- SW2 pad 1: GNDPWR -> GND
- SW3 pad 1: GNDPWR -> GND
- TP6 pad 1: GNDPWR -> GND
- TP_D1 pad 1: Net-(C17-Pad1) -> Net-(Q4-D)
- TP_S1 pad 1: Net-(C11-Pad1) -> Net-(Q4-S)
- U1 pad 1: GNDPWR -> GND
- U1 pad 10: GNDPWR -> GND
- U1 pad 12: Net-(C22-Pad2) -> Net-(U1-O0a)
- U1 pad 14: Net-(C22-Pad2) -> Net-(U1-O0a)
- U1 pad 16: Net-(C22-Pad2) -> Net-(U1-O0a)
- U1 pad 18: Net-(C22-Pad2) -> Net-(U1-O0a)
- U1 pad 19: GNDPWR -> GND
- U1 pad 3: Net-(C22-Pad2) -> Net-(U1-O0a)
- U1 pad 5: Net-(C22-Pad2) -> Net-(U1-O0a)
- U1 pad 7: Net-(C22-Pad2) -> Net-(U1-O0a)
- U1 pad 9: Net-(C22-Pad2) -> Net-(U1-O0a)
- U2 pad 2: GNDPWR -> GND
- U4 pad 4: GNDPWR -> GND
- U4 pad 7: GNDPWR -> GND
- U4 pad 8: GNDPWR -> GND
- XA1 pad 3V3: +3.3V -> +3V3
- XA1 pad A0: Net-(XA1-PadA0) -> unconnected-(XA1-PadA0)
- XA1 pad A1: Net-(XA1-PadA1) -> unconnected-(XA1-PadA1)
- XA1 pad A2: Net-(XA1-PadA2) -> unconnected-(XA1-PadA2)
- XA1 pad A3: Net-(XA1-PadA3) -> unconnected-(XA1-PadA3)
- XA1 pad A6: Net-(XA1-PadA6) -> unconnected-(XA1-PadA6)
- XA1 pad A7: Net-(XA1-PadA7) -> unconnected-(XA1-PadA7)
- XA1 pad AREF: Net-(XA1-PadAREF) -> unconnected-(XA1-PadAREF)
- XA1 pad D0: Net-(XA1-PadD0) -> unconnected-(XA1-D0_RX0-PadD0)
- XA1 pad D1: Net-(XA1-PadD1) -> unconnected-(XA1-D1_TX0-PadD1)
- XA1 pad D10: Net-(R8-Pad1) -> Net-(XA1-D10_CS)
- XA1 pad D11: Net-(R7-Pad1) -> Net-(XA1-D11_MOSI)
- XA1 pad D5: Net-(XA1-PadD5) -> unconnected-(XA1-PadD5)
- XA1 pad D6: GNDPWR -> GND
- XA1 pad D9: Net-(R9-Pad1) -> Net-(R11-Pad1)
- XA1 pad GND1: GNDPWR -> GND
- XA1 pad GND2: GNDPWR -> GND
- XA1 pad RST1: Net-(XA1-PadRST1) -> unconnected-(XA1-RESET-PadRST1)
- XA1 pad RST2: Net-(XA1-PadRST2) -> unconnected-(XA1-RESET-PadRST2)
- XA1 pad VIN: +12V -> unconnected-(XA1-PadVIN)
Routing:
- net +5V: track 189.6 -> 0.00 mm, vias 1 -> 0
- net +12V: track 150.9 -> 0.00 mm
- net FSK: track 123.4 -> 0.00 mm
- net Net-(C13-Pad1): track 103.7 -> 0.00 mm
- net SW3: track 89.6 -> 0.00 mm
- net RXSW: track 87.8 -> 0.00 mm
- net SW1: track 83.8 -> 0.00 mm, vias 1 -> 0
- net SDA: track 75.0 -> 0.00 mm
- net +3.3V: track 71.1 -> 0.00 mm
- net Net-(U1-I0a): track 66.8 -> 0.00 mm
- net RXA: track 65.2 -> 0.00 mm
- net Net-(R9-Pad1): track 64.8 -> 0.00 mm, vias 1 -> 0
- net Net-(C22-Pad2): track 64.2 -> 0.00 mm
- net SCL: track 61.6 -> 0.00 mm
- net Net-(XA1-D12_MISO): track 58.2 -> 0.00 mm
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- removed copper zone on B.Cu, net GNDPWR
- removed copper zone on F.Cu, net GNDPWR
Other:
- net class Default removed
- board text removed: "03/2022 V1.00"
- board text removed: "A"
- board text removed: "ADX - Arduino Digital Modes HF QRP Transceiver"
- board text removed: "ARDUINO USB"
- board text removed: "Band1"
- board text removed: "Band2"
- board text removed: "Band3"
- board text removed: "Band4"
- board text removed: "K"
- board text removed: "WB2CBA"
- board text removed: "WB2CBA -03/2022 V1.00"
